File: MPPT-IOBreakoutPCB.kicad_pcb (KiCad board)
At the start: 2 copper layers, 54.8 x 15.3 mm, 5 parts, among them J1 Conn_01x06, J2 Conn_01x06, J3 Conn_01x06

Commit message: fixed
Routing:
- net /CAN_L-out: track 53.0 -> 53.8 mm
